File: boards/d14b_button/d14b_button.sch (KiCad schematic (older format))
At the start: 14 parts, among them SW1 SW_PUSH, SW2 SW_PUSH, U1 STM32F030F4P6TR, U2 nRF24L01+-Module

Commit message: Quartz und LED hinzugefügt.
Parts:
- added C?: 100n, symbol C
- added C?: 10n, symbol C
- added C?: 1u, symbol C
- added C?: 4.7u, symbol C
- added C? (x2): 20p, symbol C
- added D?: LED_RCBG, symbol LED_RCBG
- added P?: CONN_02X10, symbol CONN_02X10
- added R? (x3): R, symbol R
- added X?: 8M, symbol CRYSTAL
Connections:
- wire segments 37 -> 47
Other:
- moved on the sheet: SW1, SW2

Commit message: Größerer Prozessor.
Parts:
- added C?: 200n, symbol C
- added C? (x2): 20p, symbol C
- added R?: 0, symbol R
- added U?: STM32F050C6, LQFP48, symbol STM32F050C6
- added X?: 8M, symbol CRYSTAL
Connections:
- net labels removed: +3V3
- wire segments 47 -> 53
Other:
- note removed: "TODO\n\nWandler für Eingang\nQuarz als Taktquelle\nzusätzliche Entkopplung?"
- moved on the sheet: C?, D?, P?, R?, SW1, SW2, X?

Commit message: Mittagessen
Parts:
- removed U1: STM32F030F4P6TR, Housings_SSOP:TSSOP-20_4.4x6.5mm_Pitch0.65mm, symbol STM32F030F4P6TR
- C?: value 200n -> 100n
- C? (x2): value 20p -> 10p
- X?: value 8M -> 32.768k
Connections:
- wire segments 53 -> 47
Other:
- moved on the sheet: C?
Changed lines of the file:
@@
 $EndDescr
-$Comp
-L STM32F030F4P6TR U1
-U 1 1 5480649D
-P -4000 2650
-F 0 "U1" H -5500 3550 60  0000 C CNN
-F 1 "STM32F030F4P6TR" H -2850 1750 60  0000 C CNN
-F 2 "Housings_SSOP:TSSOP-20_4.4x6.5mm_Pitch0.65mm" H -4000 2650 40  0000 C CIN
-F 3 "" H -5500 3550 60  0000 C CNN
-	1    -4000 2650
-	1    0    0    -1
-$EndComp
 $Comp
 L nRF24L01+-Module U2
@@
 	1    0    0    -1
 $EndComp
-Wire Wire Line
-	-4000 1650 -4000 1500
 Wire Wire Line
 	4750 2200 4900 2200
@@
 MISO
 Wire Wire Line
-	-4000 3600 -4000 3700
-Wire Wire Line
 	4750 2100 4900 2100
 Text GLabel 4900 2100 2    60   Input ~ 0
@@
 Text GLabel 10600 2550 2    60   Input ~ 0
 SCK
-Wire Wire Line
-	-2300 2150 -1050 2150
-Wire Wire Line
-	-1250 2050 -2300 2050
-Wire Wire Line
-	-1250 1850 -1250 2050
-Wire Wire Line
-	-1250 1850 -1050 1850
 Wire Wire Line
 	7100 1150 7200 1150
@@
 L C C?
 U 1 1 54AF99C9
-P 3500 800
-F 0 "C?" H 3500 900 40  0000 L CNN
-F 1 "100n" H 3506 715 40  0000 L CNN
-F 2 "" H 3538 650 30  0000 C CNN
-F 3 "" H 3500 800 60  0000 C CNN
-	1    3500 800
-	-1   0    0    1
+P 2650 900
+F 0 "C?" H 2650 1000 40  0000 L CNN
+F 1 "100n" H 2656 815 40  0000 L CNN
+F 2 "" H 2688 750 30  0000 C CNN
+F 3 "" H 2650 900 60  0000 C CNN
+	1    2650 900
+	1    0    0    -1
 $EndComp
 $Comp
 L C C?
 U 1 1 54AF9BEB
-P 2750 800
-F 0 "C?" H 2750 900 40  0000 L CNN
-F 1 "10n" H 2756 715 40  0000 L CNN
-F 2 "" H 2788 650 30  0000 C CNN
-F 3 "" H 2750 800 60  0000 C CNN
-	1    2750 800
-	-1   0    0    1
+P 3650 900
+F 0 "C?" H 3650 1000 40  0000 L CNN
+F 1 "10n" H 3656 815 40  0000 L CNN
+F 2 "" H 3688 750 30  0000 C CNN
+F 3 "" H 3650 900 60  0000 C CNN
+	1    3650 900
+	1    0    0    -1
 $EndComp
 $Comp
 L C C?
 U 1 1 54AF9C52
-P 2350 800
-F 0 "C?" H 2350 900 40  0000 L CNN
-F 1 "1u" H 2356 715 40  0000 L CNN
-F 2 "" H 2388 650 30  0000 C CNN
-F 3 "" H 2350 800 60  0000 C CNN
-	1    2350 800
-	-1   0    0    1
+P 4050 900
+F 0 "C?" H 4050 1000 40  0000 L CNN
+F 1 "1u" H 4056 815 40  0000 L CNN
+F 2 "" H 4088 750 30  0000 C CNN
+F 3 "" H 4050 900 60  0000 C CNN
+	1    4050 900
+	1    0    0    -1
 $EndComp
 $Comp
 L C C?
 U 1 1 54AF9CB4
-P 3800 800
-F 0 "C?" H 3800 900 40  0000 L CNN
-F 1 "4.7u" H 3806 715 40  0000 L CNN
-F 2 "" H 3838 650 30  0000 C CNN
-F 3 "" H 3800 800 60  0000 C CNN
-	1    3800 800
-	-1   0    0    1
+P 2350 900
+F 0 "C?" H 2350 1000 40  0000 L CNN
+F 1 "4.7u" H 2356 815 40  0000 L CNN
+F 2 "" H 2388 750 30  0000 C CNN
+F 3 "" H 2350 900 60  0000 C CNN
+	1    2350 900
+	1    0    0    -1
 $EndComp
 $Comp
@@
 L 3V3 #PWR?
 U 1 1 54AF9F2F
-P 3800 1000
-F 0 "#PWR?" H 3800 1100 40  0001 C CNN
-F 1 "3V3" H 3800 1125 40  0000 C CNN
-F 2 "" H 3800 1000 60  0000 C CNN
-F 3 "" H 3800 1000 60  0000 C CNN
-	1    3800 1000
-	-1   0    0    1
+P 2350 700
+F 0 "#PWR?" H 2350 800 40  0001 C CNN
+F 1 "3V3" H 2350 825 40  0000 C CNN
+F 2 "" H 2350 700 60  0000 C CNN
+F 3 "" H 2350 700 60  0000 C CNN
+	1    2350 700
+	1    0    0    -1
 $EndComp
 $Comp
 L 3V3 #PWR?
 U 1 1 54AF9F50
-P 3500 1000
-F 0 "#PWR?" H 3500 1100 40  0001 C CNN
-F 1 "3V3" H 3500 1125 40  0000 C CNN
-F 2 "" H 3500 1000 60  0000 C CNN
-F 3 "" H 3500 1000 60  0000 C CNN
-	1    3500 1000
-	-1   0    0    1
+P 2650 700
+F 0 "#PWR?" H 2650 800 40  0001 C CNN
+F 1 "3V3" H 2650 825 40  0000 C CNN
+F 2 "" H 2650 700 60  0000 C CNN
+F 3 "" H 2650 700 60  0000 C CNN
+	1    2650 700
+	1    0    0    -1
 $EndComp
 $Comp
 L 3V3 #PWR?
 U 1 1 54AF9F71
-P 2750 1000
-F 0 "#PWR?" H 2750 1100 40  0001 C CNN
-F 1 "3V3" H 2750 1125 40  0000 C CNN
-F 2 "" H 2750 1000 60  0000 C CNN
-F 3 "" H 2750 1000 60  0000 C CNN
-	1    2750 1000
-	-1   0    0    1
+P 3650 700
+F 0 "#PWR?" H 3650 800 40  0001 C CNN
+F 1 "3V3" H 3650 825 40  0000 C CNN
+F 2 "" H 3650 700 60  0000 C CNN
+F 3 "" H 3650 700 60  0000 C CNN
+	1    3650 700
+	1    0    0    -1
 $EndComp
 $Comp
 L 3V3 #PWR?
 U 1 1 54AF9F92
-P 2350 1000
-F 0 "#PWR?" H 2350 1100 40  0001 C CNN
-F 1 "3V3" H 2350 1125 40  0000 C CNN
-F 2 "" H 2350 1000 60  0000 C CNN
-F 3 "" H 2350 1000 60  0000 C CNN
-	1    2350 1000
-	-1   0    0    1
+P 4050 700
+F 0 "#PWR?" H 4050 800 40  0001 C CNN
+F 1 "3V3" H 4050 825 40  0000 C CNN
+F 2 "" H 4050 700 60  0000 C CNN
+F 3 "" H 4050 700 60  0000 C CNN
+	1    4050 700
+	1    0    0    -1
 $EndComp
 $Comp
 L GND #PWR?
 U 1 1 54AFA0D1
-P 3800 600
-F 0 "#PWR?" H 3800 600 30  0001 C CNN
-F 1 "GND" H 3800 530 30  0001 C CNN
-F 2 "" H 3800 600 60  0000 C CNN
-F 3 "" H 3800 600 60  0000 C CNN
-	1    3800 600
-	-1   0    0    1
+P 2350 1100
+F 0 "#PWR?" H 2350 1100 30  0001 C CNN
+F 1 "GND" H 2350 1030 30  0001 C CNN
+F 2 "" H 2350 1100 60  0000 C CNN
+F 3 "" H 2350 1100 60  0000 C CNN
+	1    2350 1100
+	1    0    0    -1
 $EndComp
 $Comp
 L GND #PWR?
 U 1 1 54AFA18C
-P 3500 600
-F 0 "#PWR?" H 3500 600 30  0001 C CNN
-F 1 "GND" H 3500 530 30  0001 C CNN
-F 2 "" H 3500 600 60  0000 C CNN
-F 3 "" H 3500 600 60  0000 C CNN
-	1    3500 600
-	-1   0    0    1
+P 2650 1100
+F 0 "#PWR?" H 2650 1100 30  0001 C CNN
+F 1 "GND" H 2650 1030 30  0001 C CNN
+F 2 "" H 2650 1100 60  0000 C CNN
+F 3 "" H 2650 1100 60  0000 C CNN
+	1    2650 1100
+	1    0    0    -1
 $EndComp
 $Comp
 L GND #PWR?
 U 1 1 54AFA1CD
-P 2750 600
-F 0 "#PWR?" H 2750 600 30  0001 C CNN
-F 1 "GND" H 2750 530 30  0001 C CNN
-F 2 "" H 2750 600 60  0000 C CNN
-F 3 "" H 2750 600 60  0000 C CNN
-	1    2750 600
-	-1   0    0    1
+P 3650 1100
+F 0 "#PWR?" H 3650 1100 30  0001 C CNN
+F 1 "GND" H 3650 1030 30  0001 C CNN
+F 2 "" H 3650 1100 60  0000 C CNN
+F 3 "" H 3650 1100 60  0000 C CNN
+	1    3650 1100
+	1    0    0    -1
 $EndComp
 $Comp
 L GND #PWR?
 U 1 1 54AFA1EE
-P 2350 600
-F 0 "#PWR?" H 2350 600 30  0001 C CNN
-F 1 "GND" H 2350 530 30  0001 C CNN
-F 2 "" H 2350 600 60  0000 C CNN
-F 3 "" H 2350 600 60  0000 C CNN
-	1    2350 600
-	-1   0    0    1
+P 4050 1100
+F 0 "#PWR?" H 4050 1100 30  0001 C CNN
+F 1 "GND" H 4050 1030 30  0001 C CNN
+F 2 "" H 4050 1100 60  0000 C CNN
+F 3 "" H 4050 1100 60  0000 C CNN
+	1    4050 1100
+	1    0    0    -1
 $EndComp
 $Comp
@@
 L C C?
 U 1 1 54B015E8
-P 4050 800
-F 0 "C?" H 4050 900 40  0000 L CNN
-F 1 "200n" H 4056 715 40  0000 L CNN
-F 2 "" H 4088 650 30  0000 C CNN
-F 3 "" H 4050 800 60  0000 C CNN
-	1    4050 800
-	-1   0    0    1
+P 2100 900
+F 0 "C?" H 2100 1000 40  0000 L CNN
+F 1 "100n" H 2106 815 40  0000 L CNN
+F 2 "" H 2138 750 30  0000 C CNN
+F 3 "" H 2100 900 60  0000 C CNN
+	1    2100 900
+	1    0    0    -1
 $EndComp
 $Comp
 L GND #PWR?
 U 1 1 54B01667
-P 4050 600
-F 0 "#PWR?" H 4050 600 30  0001 C CNN
-F 1 "GND" H 4050 530 30  0001 C CNN
-F 2 "" H 4050 600 60  0000 C CNN
-F 3 "" H 4050 600 60  0000 C CNN
-	1    4050 600
-	-1   0    0    1
+P 2100 1100
+F 0 "#PWR?" H 2100 1100 30  0001 C CNN
+F 1 "GND" H 2100 1030 30  0001 C CNN
+F 2 "" H 2100 1100 60  0000 C CNN
+F 3 "" H 2100 1100 60  0000 C CNN
+	1    2100 1100
+	1    0    0    -1
 $EndComp
 $Comp
 L 3V3 #PWR?
 U 1 1 54B0168E
-P 4050 1000
-F 0 "#PWR?" H 4050 1100 40  0001 C CNN
-F 1 "3V3" H 4050 1125 40  0000 C CNN
-F 2 "" H 4050 1000 60  0000 C CNN
-F 3 "" H 4050 1000 60  0000 C CNN
-	1    4050 1000
-	-1   0    0    1
+P 2100 700
+F 0 "#PWR?" H 2100 800 40  0001 C CNN
+F 1 "3V3" H 2100 825 40  0000 C CNN
+F 2 "" H 2100 700 60  0000 C CNN
+F 3 "" H 2100 700 60  0000 C CNN
+	1    2100 700
+	1    0    0    -1
 $EndComp
 Wire Wire Line
@@
 P 1000 3850
 F 0 "X?" H 1000 4000 60  0000 C CNN
-F 1 "8M" H 1000 3700 60  0000 C CNN
+F 1 "32.768k" H 1000 3700 60  0000 C CNN
 F 2 "" H 1000 3850 60  0000 C CNN
 F 3 "" H 1000 3850 60  0000 C CNN
@@
 P 800 3550
 F 0 "C?" H 800 3650 40  0000 L CNN
-F 1 "20p" H 806 3465 40  0000 L CNN
+F 1 "10p" H 806 3465 40  0000 L CNN
 F 2 "" H 838 3400 30  0000 C CNN
 F 3 "" H 800 3550 60  0000 C CNN
@@
 P 800 4150
 F 0 "C?" H 800 4250 40  0000 L CNN
-F 1 "20p" H 806 4065 40  0000 L CNN
+F 1 "10p" H 806 4065 40  0000 L CNN
 F 2 "" H 838 4000 30  0000 C CNN
 F 3 "" H 800 4150 60  0000 C CNN
