File: boards/d14b_button/d14b_button.kicad_pcb (KiCad board)
At the start: 2 copper layers, 84 x 84 mm, 65 parts, among them CON1 USB-MICRO-B, P1 CONN_02X05, P2 CONN_01X03, P3 PIEZO_BUZZ, P4 EEPROM_SPI, Q1 MOSFET_N, Q2 IRLM6402, Q3 BSS138, SW1 SW_PUSH, SW2 SW_PUSH, SW3 SW_PUSH, SW4 SW_PUSH, U1 nRF24L01+-Module, U2 STM32F030C8T6, U3 TPS61221, X1 8M, X2 32.768k

Commit message: Platine fertig - endlich :-)
Parts:
- moved JP2 2.96 mm to (125.5, 103.6)
Routing:
- net GND: track 241.1 -> 590.9 mm, vias 0 -> 8
- net +3V3: track 191.8 -> 370.7 mm, vias 2 -> 4
- net /DIV_MEAS: track 6.61 -> 119.6 mm, vias 0 -> 1
- net /MEAS_ENABLE: track 0.00 -> 46.5 mm, vias 0 -> 1
- net /SCK: track 18.1 -> 54.7 mm, vias 0 -> 2
- net Net-(JP2-Pad2): track 0.00 -> 14.5 mm
- net Net-(C16-Pad1): track 23.0 -> 29.8 mm
- net Net-(C15-Pad1): track 32.5 -> 36.9 mm
- net /ROM_HOLD: track 20.1 -> 18.2 mm
- net /VSUP_MEAS: track 75.0 -> 75.7 mm, vias 0 -> 2
- added copper zone on B.Cu, net GND
- added copper zone on F.Cu, net GND
Other:
- board text added: "Cowbus One Schalterknoten Patrick Kanzler 2015 github.com/michz/diy14bus"
