File: boards/cowbus-protoboard/periph.sch (KiCad schematic (older format))
At the start: 9 parts, among them P4 BUZ, P5 USART_DEBUG, SW1 SW1, SW2 SW2, SW3 SW3, SW4 SW4

Commit message: first version of layout for protoboard
Parts:
- removed D1: LED_RCBG, symbol LED_RCBG
- added D1: LED_RGB_reichelt, LEDs:LED_RGB_PLLC-6, symbol LED_RGB_reichelt
- added R4, R5, R6: 150, Resistors_SMD:R_0805_HandSoldering, symbol R
- added U5: LM75AD, SMD_Packages:SOIC-8-N, symbol LM75AD
- SW1, SW2, SW3, SW4: footprint (none) -> lib:Button_SMD_Schurter_LSG
Connections:
- net labels removed: LM75AD
- wire segments 41 -> 46
Changed lines of the file:
@@
 EESchema Schematic File Version 2
+LIBS:cowbus-protoboard-rescue
 LIBS:power
 LIBS:device
@@
 LIBS:nrf24l01plus-module
 LIBS:i2c
+LIBS:led_rgb_reichelt
 LIBS:cowbus-protoboard-cache
 EELAYER 25 0
@@
 F 0 "SW1" H 1500 2660 50  0000 C CNN
 F 1 "SW1" H 1350 2470 50  0000 C CNN
-F 2 "" H 1350 2550 60  0001 C CNN
+F 2 "lib:Button_SMD_Schurter_LSG" H 1350 2550 60  0001 C CNN
 F 3 "" H 1350 2550 60  0000 C CNN
 	1    1350 2550
@@
 	1350 1000 1350 2250
 $Comp
-L +3V3 #PWR042
+L +3V3 #PWR51
 U 1 1 55A697D8
 P 1350 1000
-F 0 "#PWR042" H 1350 850 50  0001 C CNN
+F 0 "#PWR51" H 1350 850 50  0001 C CNN
 F 1 "+3V3" H 1350 1140 50  0000 C CNN
 F 2 "" H 1350 1000 60  0000 C CNN
@@
 F 0 "SW2" H 2100 2660 50  0000 C CNN
 F 1 "SW2" H 1950 2470 50  0000 C CNN
-F 2 "" H 1950 2550 60  0001 C CNN
+F 2 "lib:Button_SMD_Schurter_LSG" H 1950 2550 60  0001 C CNN
 F 3 "" H 1950 2550 60  0000 C CNN
 	1    1950 2550
@@
 	1950 1000 1950 2250
 $Comp
-L +3V3 #PWR043
+L +3V3 #PWR52
 U 1 1 55A69A43
 P 1950 1000
-F 0 "#PWR043" H 1950 850 50  0001 C CNN
+F 0 "#PWR52" H 1950 850 50  0001 C CNN
 F 1 "+3V3" H 1950 1140 50  0000 C CNN
 F 2 "" H 1950 1000 60  0000 C CNN
@@
 F 0 "SW3" H 2650 2660 50  0000 C CNN
 F 1 "SW3" H 2500 2470 50  0000 C CNN
-F 2 "" H 2500 2550 60  0001 C CNN
+F 2 "lib:Button_SMD_Schurter_LSG" H 2500 2550 60  0001 C CNN
 F 3 "" H 2500 2550 60  0000 C CNN
 	1    2500 2550
@@
 	2500 1000 2500 2250
 $Comp
-L +3V3 #PWR044
+L +3V3 #PWR53
 U 1 1 55A69ACD
 P 2500 1000
-F 0 "#PWR044" H 2500 850 50  0001 C CNN
+F 0 "#PWR53" H 2500 850 50  0001 C CNN
 F 1 "+3V3" H 2500 1140 50  0000 C CNN
 F 2 "" H 2500 1000 60  0000 C CNN
@@
 F 0 "SW4" H 3250 2660 50  0000 C CNN
 F 1 "SW4" H 3100 2470 50  0000 C CNN
-F 2 "" H 3100 2550 60  0001 C CNN
+F 2 "lib:Button_SMD_Schurter_LSG" H 3100 2550 60  0001 C CNN
 F 3 "" H 3100 2550 60  0000 C CNN
 	1    3100 2550
@@
 	3100 1000 3100 2250
 $Comp
-L +3V3 #PWR045
+L +3V3 #PWR54
 U 1 1 55A69AE1
 P 3100 1000
-F 0 "#PWR045" H 3100 850 50  0001 C CNN
+F 0 "#PWR54" H 3100 850 50  0001 C CNN
 F 1 "+3V3" H 3100 1140 50  0000 C CNN
 F 2 "" H 3100 1000 60  0000 C CNN
@@
 SW_4
 $Comp
-L LED_RCBG D1
-U 1 1 55A6A030
-P 4050 2550
-F 0 "D1" H 4050 2900 50  0000 C CNN
-F 1 "LED_RCBG" H 4050 2200 50  0000 C CNN
-F 2 "" H 4050 2500 50  0001 C CNN
-F 3 "" H 4050 2500 50  0000 C CNN
-	1    4050 2550
-	0    1    1    0
-$EndComp
-Wire Wire Line
-	4050 1000 4050 2250
-$Comp
-L +3V3 #PWR046
+L +3V3 #PWR55
 U 1 1 55A6A1D5
-P 4050 1000
-F 0 "#PWR046" H 4050 850 50  0001 C CNN
-F 1 "+3V3" H 4050 1140 50  0000 C CNN
-F 2 "" H 4050 1000 60  0000 C CNN
-F 3 "" H 4050 1000 60  0000 C CNN
-	1    4050 1000
+P 3850 1000
+F 0 "#PWR55" H 3850 850 50  0001 C CNN
+F 1 "+3V3" H 3850 1140 50  0000 C CNN
+F 2 "" H 3850 1000 60  0000 C CNN
+F 3 "" H 3850 1000 60  0000 C CNN
+	1    3850 1000
 	1    0    0    -1
 $EndComp
@@
 	4750 2550 4750 1000
 $Comp
-L +3V3 #PWR047
+L +3V3 #PWR58
 U 1 1 55A7DC62
 P 4750 1000
-F 0 "#PWR047" H 4750 850 50  0001 C CNN
+F 0 "#PWR58" H 4750 850 50  0001 C CNN
 F 1 "+3V3" H 4750 1140 50  0000 C CNN
 F 2 "" H 4750 1000 60  0000 C CNN
@@
 Text HLabel 1200 4700 0    79   Input ~ 0
 BUZ
-$Comp
-L LM75AD #U048
-U 1 1 55A751D9
-P 7450 2700
-F 0 "#U048" H 7450 2700 60  0001 C CNN
-F 1 "LM75AD" H 7700 3050 60  0000 C CNN
-F 2 "" H 7450 2700 60  0000 C CNN
-F 3 "" H 7450 2700 60  0000 C CNN
-	1    7450 2700
-	1    0    0    -1
-$EndComp
 Wire Wire Line
 	7050 2500 6900 2500
@@
 	7050 2600 6900 2600
 $Comp
-L GND #PWR049
+L GND #PWR63
 U 1 1 55A7545F
 P 7450 5350
-F 0 "#PWR049" H 7450 5100 50  0001 C CNN
+F 0 "#PWR63" H 7450 5100 50  0001 C CNN
 F 1 "GND" H 7450 5200 50  0000 C CNN
 F 2 "" H 7450 5350 60  0000 C CNN
@@
 	7450 3100 7450 5350
 $Comp
-L +3V3 #PWR050
+L +3V3 #PWR62
 U 1 1 55A75598
 P 7450 1000
-F 0 "#PWR050" H 7450 850 50  0001 C CNN
+F 0 "#PWR62" H 7450 850 50  0001 C CNN
 F 1 "+3V3" H 7450 1140 50  0000 C CNN
 F 2 "" H 7450 1000 60  0000 C CNN
@@
 $EndComp
 $Comp
-L +3V3 #PWR051
+L +3V3 #PWR59
 U 1 1 55A7583B
 P 6050 1000
-F 0 "#PWR051" H 6050 850 50  0001 C CNN
+F 0 "#PWR59" H 6050 850 50  0001 C CNN
 F 1 "+3V3" H 6050 1140 50  0000 C CNN
 F 2 "" H 6050 1000 60  0000 C CNN
@@
 	6050 1000 6050 2550
 $Comp
-L GND #PWR052
+L GND #PWR60
 U 1 1 55A7591A
 P 6050 5350
-F 0 "#PWR052" H 6050 5100 50  0001 C CNN
+F 0 "#PWR60" H 6050 5100 50  0001 C CNN
 F 1 "GND" H 6050 5200 50  0000 C CNN
 F 2 "" H 6050 5350 60  0000 C CNN
@@
 	6050 2850 6050 5350
 $Comp
-L GND #PWR053
+L GND #PWR64
 U 1 1 55A75AB9
 P 8050 5350
-F 0 "#PWR053" H 8050 5100 50  0001 C CNN
+F 0 "#PWR64" H 8050 5100 50  0001 C CNN
 F 1 "GND" H 8050 5200 50  0000 C CNN
 F 2 "" H 8050 5350 60  0000 C CNN
@@
 $EndComp
 $Comp
-L +3V3 #PWR054
+L +3V3 #PWR61
 U 1 1 55A75DDC
 P 6550 1000
-F 0 "#PWR054" H 6550 850 50  0001 C CNN
+F 0 "#PWR61" H 6550 850 50  0001 C CNN
 F 1 "+3V3" H 6550 1140 50  0000 C CNN
 F 2 "" H 6550 1000 60  0000 C CNN
@@
 	9950 3250 9950 5350
 $Comp
-L GND #PWR055
+L GND #PWR65
 U 1 1 55A968F0
 P 9950 5350
-F 0 "#PWR055" H 9950 5100 50  0001 C CNN
+F 0 "#PWR65" H 9950 5100 50  0001 C CNN
 F 1 "GND" H 9950 5200 50  0000 C CNN
 F 2 "" H 9950 5350 60  0000 C CNN
@@
 Text Notes 9250 3350 2    60   ~ 0
 Belegung\nUSART-\nUSB-Adapter:\n\n3V3\nTXD\nRXD\nGND\n+5V
+$Comp
+L LM75AD U5
+U 1 1 55BB9F38
+P 7450 2700
+F 0 "U5" H 7450 2700 60  0000 C CNN
+F 1 "LM75AD" H 7700 3050 60  0000 C CNN
+F 2 "SMD_Packages:SOIC-8-N" H 7450 2700 60  0000 C CNN
+F 3 "" H 7450 2700 60  0000 C CNN
+	1    7450 2700
+	1    0    0    -1
+$EndComp
+$Comp
+L +3V3 #PWR56
+U 1 1 55BBE42A
+P 4050 1000
+F 0 "#PWR56" H 4050 850 50  0001 C CNN
+F 1 "+3V3" H 4050 1140 50  0000 C CNN
+F 2 "" H 4050 1000 60  0000 C CNN
+F 3 "" H 4050 1000 60  0000 C CNN
+	1    4050 1000
+	1    0    0    -1
+$EndComp
+$Comp
+L +3V3 #PWR57
+U 1 1 55BBE453
+P 4250 1000
+F 0 "#PWR57" H 4250 850 50  0001 C CNN
+F 1 "+3V3" H 4250 1140 50  0000 C CNN
+F 2 "" H 4250 1000 60  0000 C CNN
+F 3 "" H 4250 1000 60  0000 C CNN
+	1    4250 1000
+	1    0    0    -1
+$EndComp
+$Comp
+L R R4
+U 1 1 55BBE474
+P 3850 1700
+F 0 "R4" V 3930 1700 50  0000 C CNN
+F 1 "150" V 3850 1700 50  0000 C CNN
+F 2 "Resistors_SMD:R_0805_HandSoldering" V 3780 1700 30  0001 C CNN
+F 3 "" H 3850 1700 30  0000 C CNN
+	1    3850 1700
+	1    0    0    -1
+$EndComp
+$Comp
+L R R5
+U 1 1 55BBE4DE
+P 4050 1700
+F 0 "R5" V 4130 1700 50  0000 C CNN
+F 1 "150" V 4050 1700 50  0000 C CNN
+F 2 "Resistors_SMD:R_0805_HandSoldering" V 3980 1700 30  0001 C CNN
+F 3 "" H 4050 1700 30  0000 C CNN
+	1    4050 1700
+	1    0    0    -1
+$EndComp
+$Comp
+L R R6
+U 1 1 55BBE526
+P 4250 1700
+F 0 "R6" V 4330 1700 50  0000 C CNN
+F 1 "150" V 4250 1700 50  0000 C CNN
+F 2 "Resistors_SMD:R_0805_HandSoldering" V 4180 1700 30  0001 C CNN
+F 3 "" H 4250 1700 30  0000 C CNN
+	1    4250 1700
+	1    0    0    -1
+$EndComp
+Wire Wire Line
+	3850 1550 3850 1000
+Wire Wire Line
+	4050 1000 4050 1550
+Wire Wire Line
+	4250 1550 4250 1000
+Wire Wire Line
+	3850 2450 3850 1850
+Wire Wire Line
+	4050 1850 4050 2450
+Wire Wire Line
+	4250 2450 4250 1850
+$Comp
+L LED_RGB_reichelt D1
+U 1 1 55BB7526
+P 4050 2650
+F 0 "D1" H 4050 3075 50  0000 C CNN
+F 1 "LED_RGB_reichelt" H 4050 3000 50  0000 C CNN
+F 2 "LEDs:LED_RGB_PLLC-6" V 3650 2650 50  0000 C CNN
+F 3 "" H 4050 2600 50  0000 C CNN
+	1    4050 2650
+	0    -1   -1   0
+$EndComp
 $EndSCHEMATC
